File: PCB/MAG_ACC.kicad_sch (KiCad schematic)
At the start: 9 parts, among them U1 LSM303AH, U2 TCA39306DCUR

Commit message: Add LEDs
Parts:
- removed R8: R_200k_1%_1/16W_0402, 001-Resistors:R_0402_H0.4, symbol Resistors:R_200k_1%_1/16W_0402
- removed U2: TCA39306DCUR, 005-ICs:TCA39306DCUR, symbol ICs:TCA39306DCUR
- added R8: R_200k_1%_1/16W_0402, 001-Resistors:R_0402_H0.4, symbol 001-Resistors:R_200k_1%_1/16W_0402
- added U2: TCA39306DCUR, 005-ICs:TCA39306DCUR, symbol 005-ICs:TCA39306DCUR
Connections:
- net +1V8: now also U2.2 (VREF1)
- net +3.3V: now also R8.1
- net GND: now also U2.1 (GND)
- net LSM_SCL: now also U2.3 (SCL1)
- net LSM_SDA: now also U2.4 (SDA1)
- net SCL: now also U2.6 (SCL2)
- net SDA: now also U2.5 (SDA2)
- new net: R8.2, U2.7 (VREF2), U2.8 (EN)

Commit message: Layout start
Parts:
- removed C13: C_220nF_50V_10%_X7R_0603_H0.9, 002-Capacitors:C_0603_H0.95, symbol 002-Capacitors:C_220nF_50V_10%_X7R_0603
- removed C14: C_10uF_10V_20%_X5R_0603H0.9, 002-Capacitors:C_0603_H0.95, symbol 002-Capacitors:C_10uF_10V_20%_X5R_0603
- removed R5, R7: R_4k7_1%_1/10W_0603, 001-Resistors:R_0603_H0.55, symbol 001-Resistors:R_4k7_1%_1/10W_0603
- added C14: C_220nF_16V_10%_X7R_0402_H0.55, 002-Capacitors:C_0402_H0.55, symbol 002-Capacitors:C_220nF_16V_10%_X7R_0402
- added C30: C_2.2uF_25V_25%_X5R_0402_H0.55, 002-Capacitors:C_0402_H0.55, symbol 002-Capacitors:C_2.2uF_25V_25%_X5R_0402
- added R5, R7: R_4k7_5%_1/16W_0402, 001-Resistors:R_0402_H0.4, symbol 001-Resistors:R_4k7_5%_1/16W_0402
Connections:
- net +1V8: now also C30.1, R5.1, R7.1
- net GND: now also C14.2, C30.2
- net LSM_SCL: now also R5.2
- net LSM_SDA: now also R7.2
- net at U1.5 (C1): now also C14.1

Commit message: First layout draft
Changed lines of the file:
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@@
+	)
+	(symbol
+		(lib_id "power:PWR_FLAG")
+		(at 198.12 97.79 270)
+		(unit 1)
+		(exclude_from_sim no)
+		(in_bom yes)
+		(on_board yes)
+		(dnp no)
+		(fields_autoplaced yes)
+		(property "Reference" "#FLG02"
+			(at 200.025 97.79 0)
+			(effects
+				(font
+					(size 1.27 1.27)
+				)
+				(hide yes)
+			)
+		)
+		(property "Value" "PWR_FLAG"
+			(at 201.93 97.7899 90)
+			(effects
+				(font
+					(size 1.27 1.27)
+				)
+				(justify left)
+			)
+		)
+		(property "Footprint" ""
+			(at 198.12 97.79 0)
+			(effects
+				(font
+					(size 1.27 1.27)
+				)
+				(hide yes)
+			)
+		)
+		(property "Datasheet" "~"
+			(at 198.12 97.79 0)
+			(effects
+				(font
+					(size 1.27 1.27)
+				)
+				(hide yes)
+			)
+		)
+		(property "Description" "Special symbol for telling ERC where power comes from"
+			(at 198.12 97.79 0)
+			(effects
+				(font
+					(size 1.27 1.27)
+				)
+				(hide yes)
+			)
+		)
+		(pin "1"
+		)
+		(instances
+			(project "relativeGPS"
+				(path "/9255e348-2f0c-48d3-8a71-46491dcb1a12/0a556df8-71a3-440f-aa98-fb69e413d0a5"
+					(reference "#FLG02")
+					(unit 1)
+				)
+			)
+		)
 	)
 	(symbol

Commit message: Add TPs
Parts:
- added TP8, TP9: TP_square_1mm, 011-Misc:Testpoint_square_1mm, symbol 011-Misc:Testpoint_square_1mm
Connections:
- net LSM_SCL: now also TP8.1
- net LSM_SDA: now also TP9.1
