File: PCB/relativeGPS.kicad_pcb (KiCad board)
At the start: 4 copper layers, 65 x 65 mm, 91 parts, among them CN1 FTSH-107-01-L-DV-K-P-TR, CN2 Solder_Jumper-2_Open, CN3 TC2030-IDC, CN4 5033981892, SW1 switch_slide_2pos, SW2 EVQ-P7A01P, SW3 EVQ-P7A01P, SW4 TL3315NF160Q, U1 LSM303AH, U10 RYLR998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

Commit message: Start placing TPs
Parts:
- added TP1: TP_square_1mm, 011-Misc:Testpoint_square_1mm, F.Cu at (103.5, 122.9)
- added TP10: TP_square_1mm, 011-Misc:Testpoint_square_1mm, F.Cu at (59.0, 123.5)
- added TP11: TP_square_1mm, 011-Misc:Testpoint_square_1mm, F.Cu at (100.3, 123.0)
- added TP12: TP_square_1mm, 011-Misc:Testpoint_square_1mm, F.Cu at (51.0, 117.5)
- added TP13: TP_square_1mm, 011-Misc:Testpoint_square_1mm, F.Cu at (51.0, 119.5)
- added TP14: TP_square_1mm, 011-Misc:Testpoint_square_1mm, F.Cu at (51.0, 123.5)
- added TP15: TP_square_1mm, 011-Misc:Testpoint_square_1mm, F.Cu at (55.0, 123.5)
- added TP16: TP_square_1mm, 011-Misc:Testpoint_square_1mm, F.Cu at (53.0, 117.5)
- added TP17: TP_square_1mm, 011-Misc:Testpoint_square_1mm, F.Cu at (53.0, 119.5)
- added TP18: TP_square_1mm, 011-Misc:Testpoint_square_1mm, F.Cu at (55.0, 117.5)
- added TP19: TP_square_1mm, 011-Misc:Testpoint_square_1mm, F.Cu at (55.0, 119.5)
- added TP2: TP_square_1mm, 011-Misc:Testpoint_square_1mm, F.Cu at (115.4, 119.9)
- added TP3: TP_square_1mm, 011-Misc:Testpoint_square_1mm, F.Cu at (98.3, 123.0)
- added TP4: TP_square_1mm, 011-Misc:Testpoint_square_1mm, F.Cu at (53.0, 113.5)
- added TP5: TP_square_1mm, 011-Misc:Testpoint_square_1mm, F.Cu at (55.0, 111.5)
- added TP6: TP_square_1mm, 011-Misc:Testpoint_square_1mm, F.Cu at (55.0, 113.5)
- added TP7: TP_square_1mm, 011-Misc:Testpoint_square_1mm, F.Cu at (57.0, 111.5)
- added TP8: TP_square_1mm, 011-Misc:Testpoint_square_1mm, F.Cu at (59.0, 117.5)
- added TP9: TP_square_1mm, 011-Misc:Testpoint_square_1mm, F.Cu at (59.0, 119.5)
- U7: footprint 005-ICs:TSSOP6_SOT363-2.step -> 005-ICs:TSSOP6_SOT363-2
Connections:
- CN1 pad 1: (no net) -> unconnected-(CN1-Pad1)
- CN1 pad 10: (no net) -> unconnected-(CN1-Pad10)
- CN1 pad 2: (no net) -> unconnected-(CN1-Pad2)
- CN1 pad 9: (no net) -> unconnected-(CN1-Pad9)
Routing:
- net +3V0: track 61.9 -> 65.7 mm
- net +BATT: track 6.97 -> 9.84 mm
- net +5V: track 227.8 -> 229.5 mm
- net GND: track 145.3 -> 146.4 mm, vias 87 -> 88
