File: PCB/relativeGPS.kicad_pcb (KiCad board)
At the start: 4 copper layers, 65 x 65 mm, 110 parts, among them CN1 FTSH-107-01-L-DV-K-P-TR, CN2 Solder_Jumper-2_Open, CN3 TC2030-IDC, CN4 5033981892, SW1 switch_slide_2pos, SW2 EVQ-P7A01P, SW3 EVQ-P7A01P, SW4 TL3315NF160Q, U1 LSM303AH, U10 RYLR998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

Commit message: Finish pcb?
Parts:
- moved TP5 69.7 mm to (118.7, 83.3)
- moved TP9 69.2 mm to (108.9, 71.5)
- moved TP8 66.8 mm to (107.4, 71.5)
- moved TP7 65.1 mm to (112.5, 77.5)
- moved TP15 62.1 mm to (103.0, 84.1)
- moved TP18 56.5 mm to (103.6, 88.7)
- moved TP19 56.5 mm to (103.6, 90.7)
- moved TP4 52.8 mm to (103.4, 97.6)
- moved TP13 48.8 mm to (83.9, 83.5)
- moved TP10 48.2 mm to (82.7, 81.5)
- moved TP6 47.5 mm to (102.2, 108.6)
- moved TP12 45.2 mm to (83.9, 86.5)
- moved TP17 42.6 mm to (75.5, 83.3)
- moved TP14 39.9 mm to (90.8, 126.4)
- moved TP16 30.1 mm to (72.0, 94.2)
Routing:
- net /SD_DETECT: track 31.7 -> 43.7 mm, vias 1 -> 2
- net /MAG_ACC/LSM_SDA: track 7.90 -> 15.7 mm
- net /RYLR998_TX: track 56.1 -> 63.3 mm, vias 1 -> 2
- net /RYLR998_RX: track 53.6 -> 59.9 mm, vias 0 -> 1
- net /TESEO_RX: track 32.1 -> 36.6 mm, vias 0 -> 1
- net /GPS/3V3_TESEO_FILTERED: track 6.94 -> 10.7 mm, vias 0 -> 1
- net /TESEO_TX: track 27.8 -> 31.4 mm, vias 0 -> 1
- net /MAG_ACC/LSM_SCL: track 4.77 -> 7.47 mm
- net +3.3V_LORA: track 43.4 -> 45.7 mm
- net +1V8: track 26.7 -> 28.8 mm
- net +3.3V: track 220.0 -> 221.8 mm
- net /LED_DATA: track 27.6 -> 28.9 mm
- net /SDA: track 70.0 -> 71.3 mm
- net /SCL: track 68.3 -> 69.6 mm
- net +3.3V_GPS: track 40.2 -> 41.4 mm
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Other:
- board text added: "1V8"
- board text added: "3V"
- board text added: "3V3"
- board text added: "3V3_GPS"
- board text added: "3V3_L"
- board text added: "3V_GPS"
- board text added: "5V"
- board text added: "GND"
- board text added: "LED"
- board text added: "RX_G"
- board text added: "RX_L"
- board text added: "SCL"
- board text added: "SCL_L"
- board text added: "SD"
- board text added: "SDA"
- board text added: "SDA_L"
- board text added: "TX_G"
- board text added: "TX_L"
- board text added: "VBAT"
