File: PCB/relativeGPS.kicad_pcb (KiCad board)
At the start: 4 copper layers, 65 x 65 mm, 110 parts, among them CN1 FTSH-107-01-L-DV-K-P-TR, CN2 Solder_Jumper-2_Open, CN3 TC2030-IDC, CN4 5033981892, SW1 switch_slide_2pos, SW2 EVQ-P7A01P, SW3 EVQ-P7A01P, SW4 TL3315NF160Q, U1 LSM303AH, U10 RYLR998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

Commit message: Replace outdated inductor
Parts:
- L4: value L_4.7uH_20%_850mA_168mOhm -> L_4.7uH_20%_1.7A_120mOhm; footprint 003-Inductors:LQH3NPZ4R7MGRL -> 003-Inductors:LQH3NPZ4R7MMEL
