File: PCB/relativeGPS.kicad_sch (KiCad schematic)
At the start: 18 parts, among them CN1 FTSH-107-01-L-DV-K-P-TR, CN3 TC2030-IDC, SW2 EVQ-P7A01P, SW3 EVQ-P7A01P, SW4 TL3315NF160Q, U11 STM32L431RCT6TR, U12 ASE-8.000MHZ-L-C-T

Commit message: First layout draft
Connections:
- net 1V8_ACC_MAG_EN: now also U11.45 (PA12)
- net 3V3_RYLR_EN: now also U11.33 (PB12)
- net 3V3_TESEO_EN: now also U11.38 (PC7)
- net BUTTON_1: now also U11.21 (PA5)
- net MAG_ACC_DRDY: now also U11.34 (PB13)
- net MAG_ACC_INT1: now also U11.35 (PB14)
- net MAG_ACC_INT2: now also U11.37 (PC6)
- net SD_DETECT: now also U11.41 (PA8); no longer U11.56 (PB4)
- no-connect marks 2 -> 24
Changed lines of the file:
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@@
+	)
+	(no_connect
+		(at 259.08 69.85)
+	)
+	(no_connect
+		(at 226.06 129.54)
+	)
+	(no_connect
+		(at 259.08 128.27)
+	)
+	(no_connect
+		(at 226.06 68.58)
+	)
+	(no_connect
+		(at 259.08 77.47)
+	)
+	(no_connect
+		(at 259.08 74.93)
+	)
+	(no_connect
+		(at 226.06 101.6)
+	)
+	(no_connect
+		(at 259.08 97.79)
+	)
+	(no_connect
+		(at 226.06 96.52)
+	)
+	(no_connect
+		(at 226.06 99.06)
+	)
+	(no_connect
+		(at 259.08 59.69)
+	)
+	(no_connect
+		(at 259.08 113.03)
+	)
+	(no_connect
+		(at 226.06 71.12)
+	)
+	(no_connect
+		(at 226.06 127)
+	)
+	(no_connect
+		(at 259.08 125.73)
+	)
+	(no_connect
+		(at 259.08 115.57)
+	)
+	(no_connect
+		(at 259.08 130.81)
 	)
 	(no_connect
@@
 	(no_connect
 		(at 95.25 180.34)
+	)
+	(no_connect
+		(at 259.08 110.49)
+	)
+	(no_connect
+		(at 259.08 102.87)
+	)
+	(no_connect
+		(at 259.08 62.23)
+	)
+	(no_connect
+		(at 226.06 93.98)
+	)
+	(no_connect
+		(at 226.06 132.08)
 	)
 	(wire
@@
 	)
 	(label "1V8_ACC_MAG_EN"
-		(at 146.05 111.76 0)
+		(at 259.08 90.17 0)
 		(fields_autoplaced yes)
 		(effects
@@
 	)
 	(label "SD_DETECT"
-		(at 259.08 113.03 0)
+		(at 259.08 80.01 0)
 		(fields_autoplaced yes)
 		(effects
@@
 	)
 	(label "MAG_ACC_INT2"
-		(at 158.75 125.73 180)
+		(at 226.06 109.22 180)
 		(fields_autoplaced yes)
 		(effects
@@
 	)
 	(label "MAG_ACC_INT1"
-		(at 158.75 121.92 180)
-		(fields_autoplaced yes)
-		(effects
-			(font
-				(size 1.27 1.27)
-			)
-			(justify right bottom)
+		(at 259.08 138.43 0)
+		(fields_autoplaced yes)
+		(effects
+			(font
+				(size 1.27 1.27)
+			)
+			(justify left bottom)
 		)
 	)
 	(label "3V3_TESEO_EN"
-		(at 146.05 109.22 0)
-		(fields_autoplaced yes)
-		(effects
-			(font
-				(size 1.27 1.27)
-			)
-			(justify left bottom)
+		(at 226.06 111.76 180)
+		(fields_autoplaced yes)
+		(effects
+			(font
+				(size 1.27 1.27)
+			)
+			(justify right bottom)
 		)
 	)
@@
 	)
 	(label "BUTTON_1"
-		(at 189.23 85.09 180)
-		(fields_autoplaced yes)
-		(effects
-			(font
-				(size 1.27 1.27)
-			)
-			(justify right bottom)
+		(at 259.08 72.39 0)
+		(fields_autoplaced yes)
+		(effects
+			(font
+				(size 1.27 1.27)
+			)
+			(justify left bottom)
 		)
 	)
@@
 	)
 	(label "3V3_RYLR_EN"
-		(at 146.05 114.3 0)
+		(at 259.08 133.35 0)
 		(fields_autoplaced yes)
 		(effects
@@
 	)
 	(label "MAG_ACC_DRDY"
-		(at 158.75 129.54 180)
-		(fields_autoplaced yes)
-		(effects
-			(font
-				(size 1.27 1.27)
-			)
-			(justify right bottom)
-		)
-	)
+		(at 259.08 135.89 0)
+		(fields_autoplaced yes)
+		(effects
+			(font
+				(size 1.27 1.27)
+			)
+			(justify left bottom)
+		)
+	)

Commit message: Add TPs
Parts:
- added TP12, TP13, TP16, TP17, TP18, TP19: TP_square_1mm, 011-Misc:Testpoint_square_1mm, symbol 011-Misc:Testpoint_square_1mm
Connections:
- net RYLR998_RX: now also TP18.1
- net RYLR998_TX: now also TP19.1
- net SCL: now also TP12.1
- net SDA: now also TP13.1
- net TESEO_RX: now also TP16.1
- net TESEO_TX: now also TP17.1
