File: PCB/POWER.kicad_sch (KiCad schematic)
At the start: 32 parts, among them SW1 switch_slide_2pos, U13 MIC5330-SSYML-TR, U4 ST1S12GR, U8 TPS61222DCKR, U9 TPS79318DBVR

Commit message: Fix MIC5330 DPN
Parts:
- U13: Digikey P/N IC REG LINEAR 3.3V/3.3V 8MLF -> 576-1947-1-ND
Changed lines of the file:
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@@
 			)
 		)
-		(property "Digikey P/N" "IC REG LINEAR 3.3V/3.3V 8MLF"
+		(property "Digikey P/N" "576-1947-1-ND"
 			(at 68.326 208.534 0)
 			(effects
