File: PCB/POWER.kicad_sch (KiCad schematic)
At the start: 32 parts, among them SW1 switch_slide_2pos, U13 MIC5330-SSYML-TR, U4 ST1S12GR, U8 TPS61222DCKR, U9 TPS79318DBVR

Commit message: Replace outdated inductor
Parts:
- L4: value L_4.7uH_20%_850mA_168mOhm -> L_4.7uH_20%_1.7A_120mOhm; footprint 003-Inductors:LQH3NPZ4R7MGRL -> 003-Inductors:LQH3NPZ4R7MMEL; symbol 003-Inductors:L_4.7uH_20%_850mA_168mOhm -> 003-Inductors:L_4.7uH_20%_1.7A_120mOhm; Digikey P/N 490-15965-1-ND -> 490-LQH3NPZ4R7MMELCT-ND; Height 1 -> 1.5; Manufacturer P/N LQH3NPZ4R7MGRL -> LQH3NPZ4R7MMEL; Price 0.35 -> 0.32; Web link https://www.digikey.ch/en/products/detail/murata-electronics/LQH3NPZ4R7MGRL/6799390?s=N4IgjCBcoEwAwA4DsVQGMoDMCGAbAzgKYA0IA9lANogAsAdEgAQCtAEiALqkAOALlCACqAOwCWvAPKYAsoWz4ArgCdCIAL6kAtDFQgMkXkoUlyVEAFZOajSB2RqAGQCKrAMwA5AAqMAtsuy82FZAA -> https://www.digikey.ch/en/products/detail/murata-electronics/LQH3NPZ4R7MMEL/6800642
Changed lines of the file:
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@@
 	)
 	(symbol
-		(lib_id "003-Inductors:L_4.7uH_20%_850mA_168mOhm")
+		(lib_id "003-Inductors:L_4.7uH_20%_1.7A_120mOhm")
 		(at 49.53 85.09 0)
 		(unit 1)
@@
 			)
 		)
-		(property "Value" "L_4.7uH_20%_850mA_168mOhm"
+		(property "Value" "L_4.7uH_20%_1.7A_120mOhm"
 			(at 53.848 90.17 0)
 			(effects
@@
 			)
 		)
-		(property "Footprint" "003-Inductors:LQH3NPZ4R7MGRL"
+		(property "Footprint" "003-Inductors:LQH3NPZ4R7MMEL"
 			(at 49.53 93.98 0)
 			(effects
@@
 			)
 		)
-		(property "Datasheet" "https://search.murata.co.jp/Ceramy/image/img/P02/JELF243A-9130.pdf"
+		(property "Datasheet" "https://search.murata.co.jp/Ceramy/image/img/P02/JELF243A-9140.pdf"
 			(at 49.53 108.204 0)
 			(effects
@@
 			)
 		)
-		(property "Web link" "https://www.digikey.ch/en/products/detail/murata-electronics/LQH3NPZ4R7MGRL/6799390?s=N4IgjCBcoEwAwA4DsVQGMoDMCGAbAzgKYA0IA9lANogAsAdEgAQCtAEiALqkAOALlCACqAOwCWvAPKYAsoWz4ArgCdCIAL6kAtDFQgMkXkoUlyVEAFZOajSB2RqAGQCKrAMwA5AAqMAtsuy82FZAA"
+		(property "Web link" "https://www.digikey.ch/en/products/detail/murata-electronics/LQH3NPZ4R7MMEL/6800642"
 			(at 49.784 105.664 0)
 			(effects
@@
 			)
 		)
-		(property "Manufacturer P/N" "LQH3NPZ4R7MGRL"
+		(property "Manufacturer P/N" "LQH3NPZ4R7MMEL"
 			(at 49.53 103.632 0)
 			(effects
@@
 			)
 		)
-		(property "Digikey P/N" "490-15965-1-ND"
+		(property "Digikey P/N" "490-LQH3NPZ4R7MMELCT-ND"
 			(at 49.784 99.314 0)
 			(effects
@@
 			)
 		)
-		(property "Price" "0.35"
+		(property "Price" "0.32"
 			(at 49.784 112.268 0)
 			(effects
@@
 			)
 		)
-		(property "Height" "1"
+		(property "Height" "1.5"
 			(at 49.784 97.028 0)
 			(effects
